File: nucleo-64-MB1360/connectors.sch (KiCad schematic (older format))
At the start: 8 parts, among them CN1 Conn_02x19_Odd_Even, CN2 Conn_02x19_Odd_Even, CN3 Conn_01x08, CN4 Conn_01x10, CN5 Conn_01x06, CN6 Conn_01x08, CN7 Conn_01x02, CN8 Conn_01x02

Commit message: set position for connectors
Parts:
- CN3, CN6: footprint Connector_PinHeader_2.54mm:PinHeader_1x08_P2.54mm_Vertical -> Connector_PinSocket_2.54mm:PinSocket_1x08_P2.54mm_Vertical
- CN4: footprint Connector_PinHeader_2.54mm:PinHeader_1x10_P2.54mm_Vertical -> Connector_PinSocket_2.54mm:PinSocket_1x10_P2.54mm_Vertical
- CN5: footprint Connector_PinHeader_2.54mm:PinHeader_1x06_P2.54mm_Vertical -> Connector_PinSocket_2.54mm:PinSocket_1x06_P2.54mm_Vertical
Changed lines of the file:
@@
 F 0 "CN6" H 3200 2350 50  0000 C CNN
 F 1 "Conn_01x08" H 3130 2301 50  0001 L CNN
-F 2 "Connector_PinHeader_2.54mm:PinHeader_1x08_P2.54mm_Vertical" H 3050 2400 50  0001 C CNN
+F 2 "Connector_PinSocket_2.54mm:PinSocket_1x08_P2.54mm_Vertical" H 3050 2400 50  0001 C CNN
 F 3 "~" H 3050 2400 50  0001 C CNN
 	1    3050 2400
@@
 F 0 "CN4" H 3200 1400 50  0000 C CNN
 F 1 "Conn_01x10" H 3130 1351 50  0001 L CNN
-F 2 "Connector_PinHeader_2.54mm:PinHeader_1x10_P2.54mm_Vertical" H 3050 1450 50  0001 C CNN
+F 2 "Connector_PinSocket_2.54mm:PinSocket_1x10_P2.54mm_Vertical" H 3050 1450 50  0001 C CNN
 F 3 "~" H 3050 1450 50  0001 C CNN
 	1    3050 1450
@@
 F 0 "CN5" H 2280 2496 50  0000 L CNN
 F 1 "Conn_01x06" H 2280 2451 50  0001 L CNN
-F 2 "Connector_PinHeader_2.54mm:PinHeader_1x06_P2.54mm_Vertical" H 2200 2550 50  0001 C CNN
+F 2 "Connector_PinSocket_2.54mm:PinSocket_1x06_P2.54mm_Vertical" H 2200 2550 50  0001 C CNN
 F 3 "~" H 2200 2550 50  0001 C CNN
 	1    2200 2550
@@
 F 0 "CN3" H 2280 1696 50  0000 L CNN
 F 1 "Conn_01x08" H 2280 1651 50  0001 L CNN
-F 2 "Connector_PinHeader_2.54mm:PinHeader_1x08_P2.54mm_Vertical" H 2200 1750 50  0001 C CNN
+F 2 "Connector_PinSocket_2.54mm:PinSocket_1x08_P2.54mm_Vertical" H 2200 1750 50  0001 C CNN
 F 3 "~" H 2200 1750 50  0001 C CNN
 	1    2200 1750
@@
 Wire Wire Line
 	3250 3000 3450 3000
+Text Label 3450 3000 2    50   ~ 0
+GND
 Wire Bus Line
 	1700 3250 1700 5300
@@
 Wire Bus Line
 	3550 1100 3550 3250
-Text Label 3450 3000 2    50   ~ 0
-GND
 $EndSCHEMATC
